File: main_box/Distribution.kicad_sch (KiCad schematic)
At the start: 0 parts

Commit message: Added 5v pówer supply for independent raspberry pi power, modified the switchgear topology
Parts:
- added DB? (x8): ~, symbol din_rail_devices:Distribution_block_4_bars_04x07
Connections:
- new net +12V: DB?.8
- new net +48V: DB?.1
- new net 48V1: DB?.2
- new net 48V2: DB?.3
- new net 48V3: DB?.4
- new net 48V4: DB?.5
- new net Earth_Protective: DB?.15
- new net GND: DB?.15, DB?.22
- new net L1: DB?.2
- new net L2: DB?.3
- new net L3: DB?.4
- new net N1: DB?.9
- new net N2: DB?.10
- new net N3: DB?.11
- new net N4: DB?.12
- new net N5: DB?.13
- new net N6: DB?.14
- new net PE1: DB?.16
- new net PE2: DB?.17
- new net PE3: DB?.18
- new net gnd_1: DB?.24
- new net gnd_2: DB?.25
- new net gnd_48v: DB?.16
- new net gnd_5v: DB?.23
- new net interruptor1_Lout: DB?.1

Commit message: last changes
Parts:
- gave numbers to parts that had none: 2
Connections:
- net N6: no longer names the net of DB1.14
- net interruptor1_Lout renamed L0
Changed lines of the file:
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@@
-    )
-  )
-  (global_label "N6" (shape input) (at 97.79 64.135 90) (fields_autoplaced)
-    (effects (font (size 1.27 1.27)) (justify left))
-    (property "Intersheet References" "${INTERSHEET_REFS}" (id 0) (at 97.7106 59.1819 90)
-      (effects (font (size 1.27 1.27)) (justify left) hide)
     )
   )
@@
     )
   )
-  (global_label "interruptor1_Lout" (shape input) (at 67.31 40.64 180) (fields_autoplaced)
+  (global_label "L0" (shape input) (at 67.31 40.64 180) (fields_autoplaced)
     (effects (font (size 1.27 1.27)) (justify right))
-    (property "Intersheet References" "${INTERSHEET_REFS}" (id 0) (at 48.5683 40.7194 0)
+    (property "Intersheet References" "${INTERSHEET_REFS}" (id 0) (at 62.6593 40.5606 0)
       (effects (font (size 1.27 1.27)) (justify right) hide)
     )
@@
   (symbol (lib_id "din_rail_devices:Distribution_block_4_bars_04x07") (at 82.55 72.39 0) (unit 2)
     (in_bom yes) (on_board yes)
-    (property "Reference" "DB?" (id 0) (at 82.55 73.66 0))
+    (property "Reference" "DB1" (id 0) (at 82.55 73.66 0))
     (property "Value" "~" (id 1) (at 82.55 80.01 0)
       (effects (font (size 1.27 1.27)) hide)
@@
   (symbol (lib_id "power:+48V") (at 135.89 43.815 0) (unit 1)
     (in_bom yes) (on_board yes) (fields_autoplaced)
-    (property "Reference" "#PWR?" (id 0) (at 135.89 47.625 0)
+    (property "Reference" "#PWR04" (id 0) (at 135.89 47.625 0)
       (effects (font (size 1.27 1.27)) hide)
     )
@@
   (symbol (lib_id "din_rail_devices:Distribution_block_4_bars_04x07") (at 82.55 52.07 0) (unit 1)
     (in_bom yes) (on_board yes)
-    (property "Reference" "DB?" (id 0) (at 82.55 57.15 0))
+    (property "Reference" "DB1" (id 0) (at 82.55 57.15 0))
     (property "Value" "~" (id 1) (at 82.55 59.69 0)
       (effects (font (size 1.27 1.27)) hide)
@@
   (symbol (lib_id "din_rail_devices:Distribution_block_4_bars_04x07") (at 82.55 113.03 0) (unit 4)
     (in_bom yes) (on_board yes) (fields_autoplaced)
-    (property "Reference" "DB?" (id 0) (at 82.55 118.11 0))
+    (property "Reference" "DB1" (id 0) (at 82.55 118.11 0))
     (property "Value" "~" (id 1) (at 82.55 120.65 0)
       (effects (font (size 1.27 1.27)) hide)
@@
   (symbol (lib_id "power:GND") (at 129.54 111.76 0) (unit 1)
     (in_bom yes) (on_board yes) (fields_autoplaced)
-    (property "Reference" "#PWR?" (id 0) (at 129.54 118.11 0)
+    (property "Reference" "#PWR07" (id 0) (at 129.54 118.11 0)
       (effects (font (size 1.27 1.27)) hide)
     )
@@
   (symbol (lib_id "power:Earth_Protective") (at 57.15 90.17 0) (unit 1)
     (in_bom yes) (on_board yes) (fields_autoplaced)
-    (property "Reference" "#PWR?" (id 0) (at 63.5 96.52 0)
+    (property "Reference" "#PWR06" (id 0) (at 63.5 96.52 0)
       (effects (font (size 1.27 1.27)) hide)
     )
@@
   (symbol (lib_id "din_rail_devices:Distribution_block_4_bars_04x07") (at 151.13 73.66 0) (unit 2)
     (in_bom yes) (on_board yes)
-    (property "Reference" "DB?" (id 0) (at 151.13 74.93 0))
+    (property "Reference" "DB2" (id 0) (at 151.13 74.93 0))
     (property "Value" "~" (id 1) (at 151.13 81.28 0)
       (effects (font (size 1.27 1.27)) hide)
@@
   (symbol (lib_id "din_rail_devices:Distribution_block_4_bars_04x07") (at 82.55 93.98 0) (unit 3)
     (in_bom yes) (on_board yes) (fields_autoplaced)
-    (property "Reference" "DB?" (id 0) (at 82.55 99.06 0))
+    (property "Reference" "DB1" (id 0) (at 82.55 99.06 0))
     (property "Value" "~" (id 1) (at 82.55 101.6 0)
       (effects (font (size 1.27 1.27)) hide)
@@
   (symbol (lib_id "power:+12V") (at 135.89 66.04 0) (unit 1)
     (in_bom yes) (on_board yes) (fields_autoplaced)
-    (property "Reference" "#PWR?" (id 0) (at 135.89 69.85 0)
+    (property "Reference" "#PWR05" (id 0) (at 135.89 69.85 0)
       (effects (font (size 1.27 1.27)) hide)
     )
@@
   (symbol (lib_id "din_rail_devices:Distribution_block_4_bars_04x07") (at 151.13 53.34 0) (unit 1)
     (in_bom yes) (on_board yes)
-    (property "Reference" "DB?" (id 0) (at 151.13 58.42 0))
+    (property "Reference" "DB2" (id 0) (at 151.13 58.42 0))
     (property "Value" "~" (id 1) (at 151.13 60.96 0)
       (effects (font (size 1.27 1.27)) hide)
@@
   (symbol (lib_id "din_rail_devices:Distribution_block_4_bars_04x07") (at 151.13 114.3 0) (unit 4)
     (in_bom yes) (on_board yes) (fields_autoplaced)
-    (property "Reference" "DB?" (id 0) (at 151.13 119.38 0))
+    (property "Reference" "DB2" (id 0) (at 151.13 119.38 0))
     (property "Value" "~" (id 1) (at 151.13 121.92 0)
       (effects (font (size 1.27 1.27)) hide)
@@
   (symbol (lib_id "din_rail_devices:Distribution_block_4_bars_04x07") (at 151.13 93.98 0) (unit 3)
     (in_bom yes) (on_board yes) (fields_autoplaced)
-    (property "Reference" "DB?" (id 0) (at 151.13 99.06 0))
+    (property "Reference" "DB2" (id 0) (at 151.13 99.06 0))
     (property "Value" "~" (id 1) (at 151.13 101.6 0)
       (effects (font (size 1.27 1.27)) hide)
