File: main_box/Power_input.kicad_sch (KiCad schematic)
At the start: 0 parts

Commit message: Added 5v pówer supply for independent raspberry pi power, modified the switchgear topology
Parts:
- added CB?: differential_2P, symbol din_rail_devices:differential_2P
- added CB?: CircuitBreaker_1P, symbol Device:CircuitBreaker_1P
- added PS?: ~, symbol external_modules:power_suppy
- added PS?: power_suppy, symbol external_modules:power_suppy
Connections:
- new net: CB?.1, CB?.2
- new net +48V: PS?.7 (+Vout2)
- new net 5V_RASPI: PS?.7 (+Vout2)
- new net AC: CB?.2
- new net GND_RASPI: PS?.5 (-Vout2)
- new net L1: PS?.1 (AC/L)
- new net L2: PS?.1 (AC/L)
- new net N0: CB?.N
- new net N1: PS?.2 (AC/N)
- new net N2: PS?.2 (AC/N)
- new net NEUT: CB?.N
- new net PE1: PS?.3 (PG)
- new net PE2: PS?.3 (PG)
- new net gnd_48v: PS?.4 (-Vout1)
- new net gnd_5v: PS?.4 (-Vout1)
- new net interruptor1_Lin: CB?.1

Commit message: last changes
Parts:
- gave numbers to parts that had none: 4
Connections:
- net L1 renamed interruptor1_Lout
- net L2 renamed interruptor2_Lout
- net interruptor1_Lin renamed L0
Changed lines of the file:
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@@
+    )
+  )
+  (global_label "interruptor2_Lout" (shape input) (at 45.72 91.44 180) (fields_autoplaced)
+    (effects (font (size 1.27 1.27)) (justify right))
+    (property "Intersheet References" "${INTERSHEET_REFS}" (id 0) (at 26.9783 91.5194 0)
+      (effects (font (size 1.27 1.27)) (justify right) hide)
+    )
+  )
+  (global_label "interruptor1_Lout" (shape input) (at 45.72 59.69 180) (fields_autoplaced)
+    (effects (font (size 1.27 1.27)) (justify right))
+    (property "Intersheet References" "${INTERSHEET_REFS}" (id 0) (at 26.9783 59.7694 0)
+      (effects (font (size 1.27 1.27)) (justify right) hide)
     )
   )
@@
     )
   )
-  (global_label "L2" (shape input) (at 45.72 91.44 90) (fields_autoplaced)
-    (effects (font (size 1.27 1.27)) (justify left))
-    (property "Intersheet References" "${INTERSHEET_REFS}" (id 0) (at 45.6406 86.7893 90)
-      (effects (font (size 1.27 1.27)) (justify left) hide)
-    )
-  )
   (global_label "gnd_48v" (shape input) (at 71.12 107.95 270) (fields_autoplaced)
     (effects (font (size 1.27 1.27)) (justify right))
@@
     )
   )
-  (global_label "L1" (shape input) (at 45.72 59.69 90) (fields_autoplaced)
-    (effects (font (size 1.27 1.27)) (justify left))
-    (property "Intersheet References" "${INTERSHEET_REFS}" (id 0) (at 45.6406 55.0393 90)
-      (effects (font (size 1.27 1.27)) (justify left) hide)
-    )
-  )
   (global_label "gnd_5v" (shape input) (at 72.39 73.66 270) (fields_autoplaced)
     (effects (font (size 1.27 1.27)) (justify right))
@@
     )
   )
-  (global_label "interruptor1_Lin" (shape input) (at 80.01 41.91 90) (fields_autoplaced)
+  (global_label "L0" (shape input) (at 80.01 41.91 90) (fields_autoplaced)
     (effects (font (size 1.27 1.27)) (justify left))
-    (property "Intersheet References" "${INTERSHEET_REFS}" (id 0) (at 79.9306 24.4383 90)
+    (property "Intersheet References" "${INTERSHEET_REFS}" (id 0) (at 79.9306 37.2593 90)
       (effects (font (size 1.27 1.27)) (justify left) hide)
     )
@@
   (symbol (lib_id "power:AC") (at 31.115 36.83 0) (unit 1)
     (in_bom yes) (on_board yes) (fields_autoplaced)
-    (property "Reference" "#PWR?" (id 0) (at 31.115 39.37 0)
+    (property "Reference" "#PWR01" (id 0) (at 31.115 39.37 0)
       (effects (font (size 1.27 1.27)) hide)
     )
@@
   (symbol (lib_id "din_rail_devices:differential_2P") (at 45.085 43.18 270) (unit 1)
     (in_bom yes) (on_board yes) (fields_autoplaced)
-    (property "Reference" "CB?" (id 0) (at 49.53 28.575 90))
+    (property "Reference" "CB2" (id 0) (at 49.53 28.575 90))
     (property "Value" "differential_2P" (id 1) (at 49.53 31.115 90))
     (property "Footprint" "" (id 2) (at 42.545 52.07 0)
@@
   (symbol (lib_id "power:+48V") (at 69.85 90.17 0) (unit 1)
     (in_bom yes) (on_board yes)
-    (property "Reference" "#PWR?" (id 0) (at 69.85 93.98 0)
+    (property "Reference" "#PWR03" (id 0) (at 69.85 93.98 0)
       (effects (font (size 1.27 1.27)) hide)
     )
@@
   (symbol (lib_id "external_modules:power_suppy") (at 58.42 99.06 0) (unit 1)
     (in_bom yes) (on_board yes) (fields_autoplaced)
-    (property "Reference" "PS?" (id 0) (at 58.42 87.63 0))
+    (property "Reference" "PS2" (id 0) (at 58.42 87.63 0))
     (property "Value" "~" (id 1) (at 58.42 90.17 0))
     (property "Footprint" "" (id 2) (at 58.42 105.41 0)
@@
   (symbol (lib_id "Device:CircuitBreaker_1P") (at 69.85 41.91 270) (unit 1)
     (in_bom yes) (on_board yes) (fields_autoplaced)
-    (property "Reference" "CB?" (id 0) (at 69.85 33.655 90))
+    (property "Reference" "CB1" (id 0) (at 69.85 33.655 90))
     (property "Value" "CircuitBreaker_1P" (id 1) (at 69.85 36.195 90))
     (property "Footprint" "" (id 2) (at 69.85 41.91 0)
@@
   (symbol (lib_id "external_modules:power_suppy") (at 58.42 67.31 0) (unit 1)
     (in_bom yes) (on_board yes) (fields_autoplaced)
-    (property "Reference" "PS?" (id 0) (at 58.42 55.88 0))
+    (property "Reference" "PS1" (id 0) (at 58.42 55.88 0))
     (property "Value" "power_suppy" (id 1) (at 58.42 58.42 0))
     (property "Footprint" "" (id 2) (at 58.42 73.66 0)
@@
   (symbol (lib_id "power:NEUT") (at 26.035 42.545 0) (unit 1)
     (in_bom yes) (on_board yes)
-    (property "Reference" "#PWR?" (id 0) (at 26.035 46.355 0)
+    (property "Reference" "#PWR02" (id 0) (at 26.035 46.355 0)
       (effects (font (size 1.27 1.27)) hide)
     )
