File: main_box/Switchgear.kicad_sch (KiCad schematic)
At the start: 0 parts

Commit message: Added 5v pówer supply for independent raspberry pi power, modified the switchgear topology
Parts:
- added CB? (x2): CircuitBreaker_1P, symbol Device:CircuitBreaker_1P
- added KM?: ~, symbol din_rail_devices:Contactor_3P_right
- added LA? (x2): ~, symbol Device:Lamp
- added TB?: ~, symbol din_rail_devices:terminal_block_single
- added TB?: terminal_block_single, symbol din_rail_devices:terminal_block_single
Connections:
- new net 48V1: KM?.4
- new net 48V2: KM?.2
- new net 48v_RC: KM?.1, TB?.1
- new net 48v_hombro: KM?.3
- new net N3: LA?.1 (-)
- new net N4: KM?.A2, LA?.1 (-)
- new net gnd_2: TB?.1
- new net interruptor1_Lin: CB?.2
- new net interruptor1_Lout: CB?.1, LA?.2 (+)
- new net interruptor2_Lin: CB?.2
- new net interruptor2_Lout: CB?.1, KM?.A1, LA?.2 (+)

Commit message: last changes
Parts:
- added EMERGENCY_STOP1: CircuitBreaker_1P, symbol Device:CircuitBreaker_1P
- gave numbers to parts that had none: 7
Connections:
- net N4: no longer KM1.A2
- net interruptor2_Lout: now also EMERGENCY_STOP1.2; no longer KM1.A1
- net interruptor1_Lin renamed L1
- net interruptor2_Lin renamed L2
- new net EMERGENCY_OUT: EMERGENCY_STOP1.1, KM1.A1
- new net N5: KM1.A2
Changed lines of the file:
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@@
+    (stroke (width 0) (type default) (color 0 0 0 0))
+  )
+  (wire (pts (xy 41.91 110.49) (xy 44.45 110.49))
     (stroke (width 0) (type default) (color 0 0 0 0))
   )
@@
     (stroke (width 0) (type default) (color 0 0 0 0))
   )
+  (wire (pts (xy 59.69 110.49) (xy 65.405 110.49))
+    (stroke (width 0) (type default) (color 0 0 0 0))
+  )
   (wire (pts (xy 41.275 72.39) (xy 43.815 72.39))
     (stroke (width 0) (type default) (color 0 0 0 0))
@@
     )
   )
-  (global_label "interruptor2_Lout" (shape input) (at 153.67 66.04 270) (fields_autoplaced)
-    (effects (font (size 1.27 1.27)) (justify right))
-    (property "Intersheet References" "${INTERSHEET_REFS}" (id 0) (at 153.7494 84.7817 90)
-      (effects (font (size 1.27 1.27)) (justify right) hide)
-    )
-  )
-  (global_label "interruptor2_Lin" (shape input) (at 41.275 72.39 180) (fields_autoplaced)
-    (effects (font (size 1.27 1.27)) (justify right))
-    (property "Intersheet References" "${INTERSHEET_REFS}" (id 0) (at 23.8033 72.3106 0)
-      (effects (font (size 1.27 1.27)) (justify right) hide)
-    )
-  )
-  (global_label "N4" (shape input) (at 175.26 66.04 270) (fields_autoplaced)
+  (global_label "L2" (shape input) (at 41.275 72.39 180) (fields_autoplaced)
+    (effects (font (size 1.27 1.27)) (justify right))
+    (property "Intersheet References" "${INTERSHEET_REFS}" (id 0) (at 36.6243 72.3106 0)
+      (effects (font (size 1.27 1.27)) (justify right) hide)
+    )
+  )
+  (global_label "interruptor2_Lout" (shape input) (at 41.91 110.49 180) (fields_autoplaced)
+    (effects (font (size 1.27 1.27)) (justify right))
+    (property "Intersheet References" "${INTERSHEET_REFS}" (id 0) (at 23.1683 110.5694 0)
+      (effects (font (size 1.27 1.27)) (justify right) hide)
+    )
+  )
+  (global_label "N5" (shape input) (at 175.26 66.04 270) (fields_autoplaced)
     (effects (font (size 1.27 1.27)) (justify right))
     (property "Intersheet References" "${INTERSHEET_REFS}" (id 0) (at 175.1806 70.9931 90)
@@
     )
   )
+  (global_label "EMERGENCY_OUT" (shape input) (at 65.405 110.49 0) (fields_autoplaced)
+    (effects (font (size 1.27 1.27)) (justify left))
+    (property "Intersheet References" "${INTERSHEET_REFS}" (id 0) (at 83.5419 110.4106 0)
+      (effects (font (size 1.27 1.27)) (justify left) hide)
+    )
+  )
   (global_label "gnd_2" (shape input) (at 200.66 52.07 180) (fields_autoplaced)
     (effects (font (size 1.27 1.27)) (justify right))
@@
     )
   )
+  (global_label "EMERGENCY_OUT" (shape input) (at 153.67 66.04 180) (fields_autoplaced)
+    (effects (font (size 1.27 1.27)) (justify right))
+    (property "Intersheet References" "${INTERSHEET_REFS}" (id 0) (at 135.5331 66.1194 0)
+      (effects (font (size 1.27 1.27)) (justify right) hide)
+    )
+  )
   (global_label "interruptor1_Lout" (shape input) (at 66.675 46.355 0) (fields_autoplaced)
     (effects (font (size 1.27 1.27)) (justify left))
@@
     )
   )
-  (global_label "interruptor1_Lin" (shape input) (at 43.18 46.355 180) (fields_autoplaced)
-    (effects (font (size 1.27 1.27)) (justify right))
-    (property "Intersheet References" "${INTERSHEET_REFS}" (id 0) (at 25.7083 46.4344 0)
+  (global_label "L1" (shape input) (at 43.18 46.355 180) (fields_autoplaced)
+    (effects (font (size 1.27 1.27)) (justify right))
+    (property "Intersheet References" "${INTERSHEET_REFS}" (id 0) (at 38.5293 46.2756 0)
       (effects (font (size 1.27 1.27)) (justify right) hide)
     )
@@
   (symbol (lib_id "din_rail_devices:terminal_block_single") (at 210.82 52.07 0) (unit 1)
     (in_bom yes) (on_board yes) (fields_autoplaced)
-    (property "Reference" "TB?" (id 0) (at 216.535 52.0699 0)
+    (property "Reference" "TB2" (id 0) (at 216.535 52.0699 0)
       (effects (font (size 1.27 1.27)) (justify left))
     )
@@
   (symbol (lib_id "Device:CircuitBreaker_1P") (at 53.34 46.355 270) (unit 1)
     (in_bom yes) (on_board yes)
-    (property "Reference" "CB?" (id 0) (at 53.34 38.1 90))
+    (property "Reference" "CB3" (id 0) (at 53.34 38.1 90))
     (property "Value" "CircuitBreaker_1P" (id 1) (at 53.34 40.64 90))
     (property "Footprint" "" (id 2) (at 53.34 46.355 0)
@@
     (pin "2")
   )
+  (symbol (lib_id "Device:CircuitBreaker_1P") (at 52.07 110.49 270) (unit 1)
+    (in_bom yes) (on_board yes)
+    (property "Reference" "EMERGENCY_STOP1" (id 0) (at 52.07 102.235 90))
+    (property "Value" "CircuitBreaker_1P" (id 1) (at 52.07 104.775 90))
+    (property "Footprint" "" (id 2) (at 52.07 110.49 0)
+      (effects (font (size 1.27 1.27)) hide)
+    )
+    (property "Datasheet" "~" (id 3) (at 52.07 110.49 0)
+      (effects (font (size 1.27 1.27)) hide)
+    )
+    (pin "1")
+    (pin "2")
+  )
   (symbol (lib_id "din_rail_devices:terminal_block_single") (at 210.82 41.91 0) (unit 1)
     (in_bom yes) (on_board yes) (fields_autoplaced)
-    (property "Reference" "TB?" (id 0) (at 216.535 41.9099 0)
+    (property "Reference" "TB1" (id 0) (at 216.535 41.9099 0)
       (effects (font (size 1.27 1.27)) (justify left))
     )
@@
   (symbol (lib_id "Device:CircuitBreaker_1P") (at 51.435 72.39 270) (unit 1)
     (in_bom yes) (on_board yes)
-    (property "Reference" "CB?" (id 0) (at 51.435 64.135 90))
+    (property "Reference" "CB4" (id 0) (at 51.435 64.135 90))
     (property "Value" "CircuitBreaker_1P" (id 1) (at 51.435 66.675 90))
     (property "Footprint" "" (id 2) (at 51.435 72.39 0)
@@
   (symbol (lib_id "din_rail_devices:Contactor_3P_right") (at 165.1 48.26 270) (unit 1)
     (in_bom yes) (on_board yes) (fields_autoplaced)
-    (property "Reference" "KM?" (id 0) (at 165.1 34.925 90))
+    (property "Reference" "KM1" (id 0) (at 165.1 34.925 90))
     (property "Value" "~" (id 1) (at 165.1 37.465 90))
     (property "Footprint" "" (id 2) (at 162.56 55.88 0)
@@
   (symbol (lib_id "Device:Lamp") (at 64.135 51.435 0) (unit 1)
     (in_bom yes) (on_board yes) (fields_autoplaced)
-    (property "Reference" "LA?" (id 0) (at 67.945 50.1649 0)
+    (property "Reference" "LA1" (id 0) (at 67.945 50.1649 0)
       (effects (font (size 1.27 1.27)) (justify left))
     )
@@
   (symbol (lib_id "Device:Lamp") (at 62.23 77.47 0) (unit 1)
     (in_bom yes) (on_board yes) (fields_autoplaced)
-    (property "Reference" "LA?" (id 0) (at 66.04 76.1999 0)
-      (effects (font (size 1.27 1.27)) (justify left))
-    )
+    (property "Reference" "LA2" (id 0) (at 66.04 76.1999 0)
+      (effects (font (size 1.27 1.27)) (justify left))
+    )
