File: main_box/electronic_devices.kicad_sch (KiCad schematic)
At the start: 0 parts

Commit message: added odrive to electronic devices
Parts:
- added ODRV?: (no value), symbol external_modules:simplified_odrive
Connections:
- new net 48v_hombro: ODRV?.1 (Vin)
- new net gnd_2: ODRV?.2 (GND)
Changed lines of the file:
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@@
 (kicad_sch (version 20211123) (generator eeschema)
   (paper "A4")
+  (wire (pts (xy 85.09 120.65) (xy 85.09 123.19))
+    (stroke (width 0) (type default) (color 0 0 0 0))
+  )
+  (wire (pts (xy 87.63 120.65) (xy 87.63 123.19))
+    (stroke (width 0) (type default) (color 0 0 0 0))
+  )
+  (global_label "48v_hombro" (shape input) (at 85.09 123.19 270) (fields_autoplaced)
+    (effects (font (size 1.27 1.27)) (justify right))
+    (property "Intersheet References" "${INTERSHEET_REFS}" (id 0) (at 85.0106 137.0331 90)
+      (effects (font (size 1.27 1.27)) (justify right) hide)
+    )
+  )
+  (global_label "gnd_2" (shape input) (at 87.63 123.19 270) (fields_autoplaced)
+    (effects (font (size 1.27 1.27)) (justify right))
+    (property "Intersheet References" "${INTERSHEET_REFS}" (id 0) (at 87.7094 131.2274 90)
+      (effects (font (size 1.27 1.27)) (justify right) hide)
+    )
+  )
+  (symbol (lib_id "external_modules:simplified_odrive") (at 76.2 109.22 0) (unit 1)
+    (in_bom yes) (on_board yes) (fields_autoplaced)
+    (property "Reference" "ODRV?" (id 0) (at 79.375 25.4 0))
+    (property "Value" "" (id 1) (at 79.375 27.94 0))
+    (property "Footprint" "" (id 2) (at 76.2 55.88 0)
+      (effects (font (size 1.27 1.27)) hide)
+    )
+    (property "Datasheet" "" (id 3) (at 76.2 55.88 0)
+      (effects (font (size 1.27 1.27)) hide)
+    )
+    (pin "")
+    (pin "1")
+    (pin "10")
+    (pin "11")
+    (pin "12")
+    (pin "13")
+    (pin "14")
+    (pin "15")
+    (pin "16")
+    (pin "17")
+    (pin "18")
+    (pin "19")
+    (pin "2")
+    (pin "20")
+    (pin "21")
+    (pin "22")
+    (pin "23")
+    (pin "24")
+    (pin "25")
+    (pin "26")
+    (pin "27")
+    (pin "28")
+    (pin "29")
+    (pin "3")
+    (pin "30")
+    (pin "31")
+    (pin "32")
+    (pin "33")
+    (pin "34")
+    (pin "35")
+    (pin "36")
+    (pin "37")
+    (pin "38")
+    (pin "39")
+    (pin "4")
+    (pin "40")
+    (pin "41")
+    (pin "42")
+    (pin "5")
+    (pin "6")
+    (pin "7")
+    (pin "8")
+    (pin "9")
+  )
 )

Commit message: last changes
Parts:
- added J1: (no value), symbol Connector:Raspberry_Pi_2_3
- ODRV1: renamed from ODRV?; value (none) -> simplified_odrive
Changed lines of the file:
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@@
     )
+  )
+  (symbol (lib_id "Connector:Raspberry_Pi_2_3") (at 165.1 81.28 0) (unit 1)
+    (in_bom yes) (on_board yes) (fields_autoplaced)
+    (property "Reference" "J1" (id 0) (at 172.1994 45.72 0)
+      (effects (font (size 1.27 1.27)) (justify left))
+    )
+    (property "Value" "" (id 1) (at 172.1994 48.26 0)
+      (effects (font (size 1.27 1.27)) (justify left))
+    )
+    (property "Footprint" "" (id 2) (at 165.1 81.28 0)
+      (effects (font (size 1.27 1.27)) hide)
+    )
+    (property "Datasheet" "https://www.raspberrypi.org/documentation/hardware/raspberrypi/schematics/rpi_SCH_3bplus_1p0_reduced.pdf" (id 3) (at 165.1 81.28 0)
+      (effects (font (size 1.27 1.27)) hide)
+    )
+    (pin "1")
+    (pin "10")
+    (pin "11")
+    (pin "12")
+    (pin "13")
+    (pin "14")
+    (pin "15")
+    (pin "16")
+    (pin "17")
+    (pin "18")
+    (pin "19")
+    (pin "2")
+    (pin "20")
+    (pin "21")
+    (pin "22")
+    (pin "23")
+    (pin "24")
+    (pin "25")
+    (pin "26")
+    (pin "27")
+    (pin "28")
+    (pin "29")
+    (pin "3")
+    (pin "30")
+    (pin "31")
+    (pin "32")
+    (pin "33")
+    (pin "34")
+    (pin "35")
+    (pin "36")
+    (pin "37")
+    (pin "38")
+    (pin "39")
+    (pin "4")
+    (pin "40")
+    (pin "5")
+    (pin "6")
+    (pin "7")
+    (pin "8")
+    (pin "9")
   )
   (symbol (lib_id "external_modules:simplified_odrive") (at 76.2 109.22 0) (unit 1)
     (in_bom yes) (on_board yes) (fields_autoplaced)
-    (property "Reference" "ODRV?" (id 0) (at 79.375 25.4 0))
-    (property "Value" "" (id 1) (at 79.375 27.94 0))
+    (property "Reference" "ODRV1" (id 0) (at 79.375 25.4 0))
+    (property "Value" "simplified_odrive" (id 1) (at 79.375 27.94 0))
     (property "Footprint" "" (id 2) (at 76.2 55.88 0)
       (effects (font (size 1.27 1.27)) hide)
