File: pullup_array_odrive/pullup_array_odrive.kicad_sch (KiCad schematic)
At the start: 26 parts, among them J2 2.54mm header, J3 2.54mm header, J4 2.54mm header, J5 2.54mm header, J6 2.54mm header, J7 2.54mm header, J8 2.54mm header

Commit message: last changes
Parts:
- CAN1: value (none) -> 2.54mm header
- D1, D2, D3, D4, D5, D6, D7: footprint (none) -> Diode_SMD:D_0805_2012Metric_Pad1.15x1.40mm_HandSolder
- D8: value (none) -> R; footprint (none) -> Diode_SMD:D_0805_2012Metric_Pad1.15x1.40mm_HandSolder
- J1: value (none) -> 2.54mm header; footprint (none) -> Connector_PinSocket_2.54mm:PinSocket_1x02_P2.54mm_Vertical
- J2, J3, J4: footprint (none) -> Connector_PinSocket_2.54mm:PinSocket_1x02_P2.54mm_Vertical
- J5, J6, J7, J8: footprint TerminalBlock:TerminalBlock_bornier-2_P5.08mm -> (none)
- J9: value (none) -> Conn_01x20_Male; footprint (none) -> Connector_PinSocket_2.54mm:PinSocket_1x20_P2.54mm_Vertical
- R1, R2, R3, R4, R5, R6, R7: footprint (none) -> Resistor_SMD:R_0805_2012Metric_Pad1.20x1.40mm_HandSolder
- R8: value (none) -> 1k; footprint (none) -> Resistor_SMD:R_0805_2012Metric_Pad1.20x1.40mm_HandSolder
Connections:
- net +3V3: now also J5.1 (Pin_1), J6.1 (Pin_1), J7.1 (Pin_1), J8.1 (Pin_1); no longer J5.2 (Pin_2), J6.2 (Pin_2), J7.2 (Pin_2), J8.2 (Pin_2)
- net at D8.1 (K), J9.3 (Pin_3): now also J8.2 (Pin_2); no longer J8.1 (Pin_1)
- net at D6.1 (K), J9.5 (Pin_5): now also J6.2 (Pin_2); no longer J6.1 (Pin_1)
- net at D7.1 (K), J9.4 (Pin_4): now also J7.2 (Pin_2); no longer J7.1 (Pin_1)
- net at D5.1 (K), J9.6 (Pin_6): now also J5.2 (Pin_2); no longer J5.1 (Pin_1)
Other:
- moved on the sheet: J5, J6, J7, J8
