File: pullup_array_odrive/pullup_array_odrive.kicad_sch (KiCad schematic)
At the start: 26 parts, among them J2 2.54mm header, J3 2.54mm header, J4 2.54mm header, J5 2.54mm header, J6 2.54mm header, J7 2.54mm header, J8 2.54mm header

Commit message: finished encoder pcb
Parts:
- CAN1: value (none) -> 2.54mm header; footprint (none) -> TerminalBlock:TerminalBlock_bornier-2_P5.08mm
- D1, D2, D3, D4, D5, D6, D7: footprint (none) -> Diode_SMD:D_0805_2012Metric_Pad1.15x1.40mm_HandSolder
- D8: value (none) -> R; footprint (none) -> Diode_SMD:D_0805_2012Metric_Pad1.15x1.40mm_HandSolder
- J1: value (none) -> 2.54mm header; footprint (none) -> Connector_PinSocket_2.54mm:PinSocket_1x02_P2.54mm_Vertical
- J2, J3, J4: footprint (none) -> Connector_PinSocket_2.54mm:PinSocket_1x02_P2.54mm_Vertical
- J9: value (none) -> Conn_01x20_Male; footprint (none) -> Connector_PinSocket_2.54mm:PinSocket_1x20_P2.54mm_Vertical
- R1, R2, R3, R4, R5, R6, R7: footprint (none) -> Resistor_SMD:R_0805_2012Metric_Pad1.20x1.40mm_HandSolder
- R8: value (none) -> 1k; footprint (none) -> Resistor_SMD:R_0805_2012Metric_Pad1.20x1.40mm_HandSolder
