File: differential_encoder_encoder/differential_encoder_encoder.kicad_sch (KiCad schematic)
At the start: 13 parts, among them J101 RJ45_LED_Shielded, J102 Conn_02x08_Odd_Even, U101 MAX489E, U102 MAX489E, U103 MAX489E

Commit message: tentative odrive positioning
Parts:
- J101: footprint Connector_RJ:RJ45_Wuerth_7499010121A_Horizontal -> Connector_RJ:RJ45_Amphenol_RJHSE538X
- U101, U102, U103: footprint Package_SO:SO-16_3.9x9.9mm_P1.27mm -> Package_SO:SO-14_3.9x8.65mm_P1.27mm
Changed lines of the file:
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@@
       (effects (font (size 1.27 1.27)) (justify left))
     )
-    (property "Footprint" "Package_SO:SO-16_3.9x9.9mm_P1.27mm" (at 135.89 121.92 0)
+    (property "Footprint" "Package_SO:SO-14_3.9x8.65mm_P1.27mm" (at 135.89 121.92 0)
       (effects (font (size 1.27 1.27)) hide)
     )
@@
       (effects (font (size 1.27 1.27)) (justify left))
     )
-    (property "Footprint" "Package_SO:SO-16_3.9x9.9mm_P1.27mm" (at 133.35 165.1 0)
+    (property "Footprint" "Package_SO:SO-14_3.9x8.65mm_P1.27mm" (at 133.35 165.1 0)
       (effects (font (size 1.27 1.27)) hide)
     )
@@
       (effects (font (size 1.27 1.27)))
     )
-    (property "Footprint" "Connector_RJ:RJ45_Wuerth_7499010121A_Horizontal" (at 231.14 86.995 90)
+    (property "Footprint" "Connector_RJ:RJ45_Amphenol_RJHSE538X" (at 231.14 86.995 90)
       (effects (font (size 1.27 1.27)) hide)
     )
@@
       (effects (font (size 1.27 1.27)) (justify left))
     )
-    (property "Footprint" "Package_SO:SO-16_3.9x9.9mm_P1.27mm" (at 134.62 78.74 0)
-      (effects (font (size 1.27 1.27)) hide)
-    )
+    (property "Footprint" "Package_SO:SO-14_3.9x8.65mm_P1.27mm" (at 134.62 78.74 0)
+      (effects (font (size 1.27 1.27)) hide)
+    )
